Commit message: refine

File: src/urdf_tutorial/urdf/robot_1.xacro (robot description, xacro)
@@ -1,9 +1,9 @@
 <?xml version="1.0"?>
-<robot xmlns:xacro="http://ros.org/wiki/xacro" name="urdf_test">
+<robot xmlns:xacro="http://ros.org/wiki/xacro" name="urdf_test" >
     <!-- BASE -->
     <link name="base_link">
     </link>
     <!-- BODY LINK -->
-    <joint name="body_joint" type="fixed"> <!-- 'joink'를 'joint'로 수정 -->
+    <joint name="body_joint" type="fixed">
         <parent link="base_link"/>
         <child link="body"/>
