Commit message: 카메라 연결

File: src/week5_model/urdf/hose_robot2.urdf.xacro (robot description, xacro)
@@ -2,5 +2,5 @@
 <robot xmlns:xacro="http://www.ros.org/wiki/xacro" name="hose_plate_waffle_combined">
   <!-- TurtleBot3 Waffle 로드 -->
-  <xacro:include filename="$./turtlebot3_waffle_pi.urdf.xacro"/>
+  <xacro:include filename="./turtlebot3_waffle_pi.urdf.xacro"/>
   <!-- hose_plate 정의 -->
   <material name="hose_plate_light_black">
@@ -28,10 +28,10 @@
     </collision>
   </link>
-  <joint name="top_joint" type="fixed">
+  <joint name="top_joint" type="prismatic">
     <parent link="hose_plate_base_link"/>
     <child link="top_link"/>
-    <origin rpy="0 0 0" xyz="0 0.1 0.02"/>
-    <axis xyz="0 0 1"/>
-    <!-- <limit lower="0" upper="0.02" effort="1000" velocity="0.5"/> -->
+    <origin rpy="0 0 0" xyz="0 -0.1 0.02"/>
+    <axis xyz="0 0 1"/> <!-- z축 방향으로 선형 이동 -->
+    <limit lower="0.0" upper="0.07" effort="50.0" velocity="0.035"/>
   </joint>
   <link name="top_link">
@@ -50,3 +50,14 @@
     </collision>
   </link>
+    <!-- Transmission 설정 -->
+  <transmission name="top_joint_trans">
+    <type>transmission_interface/SimpleTransmission</type>
+    <joint name="top_joint">
+      <hardwareInterface>EffortJointInterface</hardwareInterface>
+    </joint>
+    <actuator name="motor_top">
+      <hardwareInterface>EffortJointInterface</hardwareInterface>
+      <mechanicalReduction>1</mechanicalReduction>
+    </actuator>
+  </transmission>
 </robot>

File: src/week5_model/urdf/turtlebot3_waffle_pi.urdf.xacro (robot description, xacro)
@@ -2,5 +2,5 @@
 <robot name="turtlebot3_waffle_pi" xmlns:xacro="http://ros.org/wiki/xacro">
   <xacro:include filename="$(find turtlebot3_description)/urdf/common_properties.xacro"/>
-  <xacro:include filename="$(find turtlebot3_description)/urdf/urtlebot3_waffle_pi.gazebo.xacro"/>
+  <xacro:include filename="$(find turtlebot3_description)/urdf/turtlebot3_waffle_pi.gazebo.xacro"/>
   <link name="base_footprint"/>
   <joint name="base_joint" type="fixed">
